File: burner.kicad_pcb (KiCad board)
At the start: 2 copper layers, 118.8 x 58.4 mm, 76 parts, among them IC1 MAX6675, IC2 MAX6675, J1 MCU_ISP, J12 USB_A, J13 FTDI, J14 ENCODER, J2 220V_INPUT, J3 5V_INPUT, J4 BURNER2, J5 BURNER1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

Commit message: update
Other:
- net class Default removed
